Commit message: 机械臂movelt 并可视化

File: src/r2_arm_control/urdf/r2_arm.urdf.xacro (robot description, xacro)
@@ -11,7 +11,13 @@
   <xacro:property name="shoulder_zero_offset_rad" value="${arm.get('shoulder_zero_offset_rad', 0.0)}"/>
   <xacro:property name="elbow_zero_offset_rad" value="${arm.get('elbow_zero_offset_rad', 0.0)}"/>
+  <xacro:property name="shoulder_mit_kp" value="${arm.get('kp_joint0', 0.0)}"/>
+  <xacro:property name="shoulder_mit_kd" value="${arm.get('kd_joint0', 0.0)}"/>
+  <xacro:property name="shoulder_mit_ff" value="${arm.get('feedforward_joint0', 0.0)}"/>
+  <xacro:property name="elbow_mit_kp" value="${arm.get('kp_joint1', 0.0)}"/>
+  <xacro:property name="elbow_mit_kd" value="${arm.get('kd_joint1', 0.0)}"/>
+  <xacro:property name="elbow_mit_ff" value="${arm.get('feedforward_joint1', 0.0)}"/>
   <link name="base_link">
     <visual>
-      <origin xyz="0 0 0" rpy="0 0 0"/>
+      <origin xyz="0 0 -0.06" rpy="0 0 0"/>
       <geometry>
         <box size="0.12 0.12 0.12"/>
@@ -21,4 +27,10 @@
       </material>
     </visual>
+    <collision>
+      <origin xyz="0 0 -0.06" rpy="0 0 0"/>
+      <geometry>
+        <box size="0.12 0.12 0.12"/>
+      </geometry>
+    </collision>
   </link>
   <link name="upper_arm_link">
@@ -32,4 +44,10 @@
       </material>
     </visual>
+    <collision>
+      <origin xyz="0 0 ${d1 / 2.0}" rpy="0 0 0"/>
+      <geometry>
+        <box size="0.04 0.04 ${d1}"/>
+      </geometry>
+    </collision>
   </link>
   <link name="forearm_link">
@@ -43,4 +61,10 @@
       </material>
     </visual>
+    <collision>
+      <origin xyz="${d2 / 2.0} 0 0" rpy="0 0 0"/>
+      <geometry>
+        <box size="${d2} 0.03 0.03"/>
+      </geometry>
+    </collision>
   </link>
   <link name="tool_link">
@@ -54,9 +78,15 @@
       </material>
     </visual>
+    <collision>
+      <origin xyz="0 0 0" rpy="0 0 0"/>
+      <geometry>
+        <sphere radius="0.02"/>
+      </geometry>
+    </collision>
   </link>
   <joint name="shoulder_joint" type="revolute">
     <parent link="base_link"/>
     <child link="upper_arm_link"/>
-    <origin xyz="0 0 0.06" rpy="0 0 0"/>
+    <origin xyz="0 0 0" rpy="0 0 0"/>
     <axis xyz="0 1 0"/>
     <limit
@@ -98,9 +128,9 @@
       <param name="motor_sign">${shoulder_motor_sign}</param>
       <param name="zero_offset_rad">${shoulder_zero_offset_rad}</param>
-      <command_interface name="position_des"/>
-      <command_interface name="velocity_des"/>
-      <command_interface name="kp"/>
-      <command_interface name="kd"/>
-      <command_interface name="feedforward"/>
+      <param name="mit_kp">${shoulder_mit_kp}</param>
+      <param name="mit_kd">${shoulder_mit_kd}</param>
+      <param name="mit_feedforward">${shoulder_mit_ff}</param>
+      <command_interface name="position"/>
+      <command_interface name="velocity"/>
       <state_interface name="position"/>
       <state_interface name="velocity"/>
@@ -115,9 +145,9 @@
       <param name="motor_sign">${elbow_motor_sign}</param>
       <param name="zero_offset_rad">${elbow_zero_offset_rad}</param>
-      <command_interface name="position_des"/>
-      <command_interface name="velocity_des"/>
-      <command_interface name="kp"/>
-      <command_interface name="kd"/>
-      <command_interface name="feedforward"/>
+      <param name="mit_kp">${elbow_mit_kp}</param>
+      <param name="mit_kd">${elbow_mit_kd}</param>
+      <param name="mit_feedforward">${elbow_mit_ff}</param>
+      <command_interface name="position"/>
+      <command_interface name="velocity"/>
       <state_interface name="position"/>
       <state_interface name="velocity"/>

Commit message: 运动学修正 电机发送修正角度

File: src/r2_arm_control/urdf/r2_arm.urdf.xacro (robot description, xacro)
@@ -7,8 +7,12 @@
   <xacro:property name="d1" value="${arm['d1']}"/>
   <xacro:property name="d2" value="${arm['d2']}"/>
+  <xacro:property name="forearm_mount_offset_rad" value="${arm.get('forearm_mount_offset_rad', 0.0)}"/>
   <xacro:property name="shoulder_motor_sign" value="${arm.get('shoulder_motor_sign', arm.get('joint0_sign', 1.0))}"/>
   <xacro:property name="elbow_motor_sign" value="${arm.get('elbow_motor_sign', arm.get('joint1_sign', 1.0))}"/>
   <xacro:property name="shoulder_zero_offset_rad" value="${arm.get('shoulder_zero_offset_rad', 0.0)}"/>
   <xacro:property name="elbow_zero_offset_rad" value="${arm.get('elbow_zero_offset_rad', 0.0)}"/>
+  <xacro:property name="shoulder_transmission_ratio" value="${arm.get('shoulder_transmission_ratio', 1.0)}"/>
+  <xacro:property name="elbow_transmission_ratio" value="${arm.get('elbow_transmission_ratio', 1.0)}"/>
+  <xacro:property name="elbow_absolute_reference_joint" value="${arm.get('elbow_absolute_reference_joint', '')}"/>
   <xacro:property name="shoulder_mit_kp" value="${arm.get('kp_joint0', 0.0)}"/>
   <xacro:property name="shoulder_mit_kd" value="${arm.get('kd_joint0', 0.0)}"/>
@@ -99,5 +103,5 @@
     <parent link="upper_arm_link"/>
     <child link="forearm_link"/>
-    <origin xyz="0 0 ${d1}" rpy="0 0 0"/>
+    <origin xyz="0 0 ${d1}" rpy="0 ${forearm_mount_offset_rad} 0"/>
     <axis xyz="0 1 0"/>
     <limit
@@ -128,4 +132,5 @@
       <param name="motor_sign">${shoulder_motor_sign}</param>
       <param name="zero_offset_rad">${shoulder_zero_offset_rad}</param>
+      <param name="transmission_ratio">${shoulder_transmission_ratio}</param>
       <param name="mit_kp">${shoulder_mit_kp}</param>
       <param name="mit_kd">${shoulder_mit_kd}</param>
@@ -145,4 +150,6 @@
       <param name="motor_sign">${elbow_motor_sign}</param>
       <param name="zero_offset_rad">${elbow_zero_offset_rad}</param>
+      <param name="transmission_ratio">${elbow_transmission_ratio}</param>
+      <param name="absolute_reference_joint">${elbow_absolute_reference_joint}</param>
       <param name="mit_kp">${elbow_mit_kp}</param>
       <param name="mit_kd">${elbow_mit_kd}</param>

Commit message: 优化机械臂状态机继电器保持逻辑与终端状态显示

File: src/r2_arm_control/urdf/r2_arm.urdf.xacro (robot description, xacro)
@@ -15,4 +15,6 @@
   <xacro:property name="elbow_transmission_ratio" value="${arm.get('elbow_transmission_ratio', 1.0)}"/>
   <xacro:property name="elbow_absolute_reference_joint" value="${arm.get('elbow_absolute_reference_joint', '')}"/>
+  <xacro:property name="elbow_rel_min" value="${arm.get('elbow_rel_min', -1.3962634)}"/>
+  <xacro:property name="elbow_rel_max" value="${arm.get('elbow_rel_max', 1.3962634)}"/>
   <xacro:property name="shoulder_mit_kp" value="${arm.get('kp_joint0', 0.0)}"/>
   <xacro:property name="shoulder_mit_kd" value="${arm.get('kd_joint0', 0.0)}"/>
@@ -106,6 +108,6 @@
     <axis xyz="0 1 0"/>
     <limit
-      lower="${arm['q2_min']}"
-      upper="${arm['q2_max']}"
+      lower="${elbow_rel_min}"
+      upper="${elbow_rel_max}"
       effort="30.0"
       velocity="2.0"/>
@@ -138,4 +140,6 @@
       <param name="zero_offset_rad">${shoulder_zero_offset_rad}</param>
       <param name="transmission_ratio">${shoulder_transmission_ratio}</param>
+      <param name="position_min">${arm['q1_min']}</param>
+      <param name="position_max">${arm['q1_max']}</param>
       <param name="mit_kp">${shoulder_mit_kp}</param>
       <param name="mit_kd">${shoulder_mit_kd}</param>
@@ -160,4 +164,6 @@
       <param name="transmission_ratio">${elbow_transmission_ratio}</param>
       <param name="absolute_reference_joint">${elbow_absolute_reference_joint}</param>
+      <param name="position_min">${elbow_rel_min}</param>
+      <param name="position_max">${elbow_rel_max}</param>
       <param name="mit_kp">${elbow_mit_kp}</param>
       <param name="mit_kd">${elbow_mit_kd}</param>
